File: Electronix/ps2_com_ps2.brd (EAGLE design)
At the start: 33.1 x 51.8 mm, 16 parts, among them IC1 MAX232, IC2 TINY13-20PU, X2 22-27-2041-04

Commit message: Add files via upload
Parts:
- C1, C2, C3, C4, C5, C6: value 0.1 -> 1.0
Changed lines of the file:
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@@
 </autorouter>
 <elements>
-<element name="C1" library="rcl" library_urn="urn:adsk.eagle:library:334" package="C025-025X050" package3d_urn="urn:adsk.eagle:package:23629/2" value="0.1" x="8.89" y="46.99" smashed="yes" rot="R180">
+<element name="C1" library="rcl" library_urn="urn:adsk.eagle:library:334" package="C025-025X050" package3d_urn="urn:adsk.eagle:package:23629/2" value="1.0" x="8.89" y="46.99" smashed="yes" rot="R180">
 <attribute name="NAME" x="6.096" y="49.276" size="1.27" layer="25" ratio="10" rot="R180"/>
 <attribute name="POPULARITY" value="65" x="-6.35" y="88.9" size="1.778" layer="27" rot="R180" display="off"/>
@@
 <attribute name="VALUE" x="11.176" y="49.784" size="1.27" layer="27" ratio="10" rot="R180"/>
 </element>
-<element name="C2" library="rcl" library_urn="urn:adsk.eagle:library:334" package="C025-025X050" package3d_urn="urn:adsk.eagle:package:23629/2" value="0.1" x="13.97" y="69.85" smashed="yes" rot="R180">
+<element name="C2" library="rcl" library_urn="urn:adsk.eagle:library:334" package="C025-025X050" package3d_urn="urn:adsk.eagle:package:23629/2" value="1.0" x="13.97" y="69.85" smashed="yes" rot="R180">
 <attribute name="NAME" x="11.176" y="72.136" size="1.27" layer="25" ratio="10" rot="R180"/>
 <attribute name="POPULARITY" value="65" x="-7.62" y="111.76" size="1.778" layer="27" rot="R180" display="off"/>
@@
 <attribute name="VALUE" x="16.256" y="72.644" size="1.27" layer="27" ratio="10" rot="R180"/>
 </element>
-<element name="C3" library="rcl" library_urn="urn:adsk.eagle:library:334" package="C025-025X050" package3d_urn="urn:adsk.eagle:package:23629/2" value="0.1" x="7.62" y="63.5" smashed="yes" rot="R90">
+<element name="C3" library="rcl" library_urn="urn:adsk.eagle:library:334" package="C025-025X050" package3d_urn="urn:adsk.eagle:package:23629/2" value="1.0" x="7.62" y="63.5" smashed="yes" rot="R90">
 <attribute name="NAME" x="6.096" y="61.214" size="1.27" layer="25" ratio="10" rot="R90"/>
 <attribute name="POPULARITY" value="65" x="49.53" y="91.44" size="1.778" layer="27" rot="R90" display="off"/>
@@
 <attribute name="VALUE" x="10.414" y="61.214" size="1.27" layer="27" ratio="10" rot="R90"/>
 </element>
-<element name="C4" library="rcl" library_urn="urn:adsk.eagle:library:334" package="C025-025X050" package3d_urn="urn:adsk.eagle:package:23629/2" value="0.1" x="7.62" y="58.42" smashed="yes" rot="R270">
+<element name="C4" library="rcl" library_urn="urn:adsk.eagle:library:334" package="C025-025X050" package3d_urn="urn:adsk.eagle:package:23629/2" value="1.0" x="7.62" y="58.42" smashed="yes" rot="R270">
 <attribute name="NAME" x="4.826" y="58.039" size="1.27" layer="25" ratio="10" rot="R270"/>
 <attribute name="POPULARITY" value="65" x="-34.29" y="24.13" size="1.778" layer="27" rot="R270" display="off"/>
@@
 <attribute name="VALUE" x="4.826" y="60.706" size="1.27" layer="27" ratio="10" rot="R270"/>
 </element>
-<element name="C5" library="rcl" library_urn="urn:adsk.eagle:library:334" package="C025-025X050" package3d_urn="urn:adsk.eagle:package:23629/2" value="0.1" x="17.78" y="45.72" smashed="yes" rot="R90">
+<element name="C5" library="rcl" library_urn="urn:adsk.eagle:library:334" package="C025-025X050" package3d_urn="urn:adsk.eagle:package:23629/2" value="1.0" x="17.78" y="45.72" smashed="yes" rot="R90">
 <attribute name="NAME" x="16.256" y="44.704" size="1.27" layer="25" ratio="10" rot="R90"/>
 <attribute name="POPULARITY" value="65" x="59.69" y="86.36" size="1.778" layer="27" rot="R90" display="off"/>
@@
 <attribute name="VALUE" x="20.574" y="43.434" size="1.27" layer="27" ratio="10" rot="R90"/>
 </element>
-<element name="C6" library="rcl" library_urn="urn:adsk.eagle:library:334" package="C025-025X050" package3d_urn="urn:adsk.eagle:package:23629/2" value="0.1" x="20.32" y="66.04" smashed="yes" rot="R270">
+<element name="C6" library="rcl" library_urn="urn:adsk.eagle:library:334" package="C025-025X050" package3d_urn="urn:adsk.eagle:package:23629/2" value="1.0" x="20.32" y="66.04" smashed="yes" rot="R270">
 <attribute name="NAME" x="21.844" y="68.326" size="1.27" layer="25" ratio="10" rot="R270"/>
 <attribute name="POPULARITY" value="65" x="-21.59" y="19.05" size="1.778" layer="27" rot="R270" display="off"/>
